Commit message: New version_1

File: src/youbot_perception/urdf/youbot_task.urdf.xacro (robot description, xacro)
@@ -60,10 +60,15 @@
     </inertial>
   </link>
-  <!-- Камера на высоте ~0.30 м над платформой, у переднего (-X) края,
-       наклон вниз ~35° (pitch=0.6 рад), смотрит по -X (yaw=pi). -->
+  <!-- Геометрия как на реальном роботе: рука манипулятора по +X (см. arm
+       origin выше, xyz=0.143), а КАМЕРА — спереди с ПРОТИВОПОЛОЖНОЙ стороны,
+       т.е. по -X. Камера по центру (y=0), на стойке ~45 см от пола; base_link
+       выше пола на ~0.14 м => над base_link ~0.31 м. Смотрит вперёд (-X) и
+       вниз на пол: yaw=pi (разворот в -X), pitch=0.7 (наклон вниз ~40°).
+       Это «перёд» робота для зрения; рука берёт кубик после разворота базы
+       (см. position_for_grasp в pick_place_mission.py). -->
   <joint name="usb_cam_joint" type="fixed">
     <parent link="plate_link"/>
     <child link="usb_cam_link"/>
-    <origin xyz="-0.20 0.0 0.30" rpy="0 0.6 3.14159"/>
+    <origin xyz="-0.20 0.0 0.31" rpy="0 0.7 3.14159"/>
   </joint>
   <!-- Оптический кадр камеры (REP-103: z вперёд, x вправо, y вниз) -->
